File: kicad/bluz_v1/bluz_v1.kicad_sch (KiCad schematic)
At the start: 62 parts, among them J1 USB_B_Micro, J11 Conn, J12 BTAnt, J2 Conn, J3 Conn, J4 Conn, J5 Conn, J6 Conn, J7 Conn, J8 Conn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

Commit message: изменено:      Documents/BluZ.png 	изменено:      kicad/bluz_v1/bluz_v1.kicad_pcb 	изменено:      kicad/bluz_v1/bluz_v1.kicad_prl 	изменено:      kicad/bluz_v1/bluz_v1.kicad_pro 	изменено:      kicad/bluz_v1/bluz_v1.kicad_sch 	изменено:      kicad/bluz_v1/fp-info-cache
Parts:
- C1, C11, C14, C17, C2, C3, C5, C6, C7: value C -> 4.7u
- C10, C13, C4, C8: value C -> 10u
- C12: value C -> .1
- D2: value LED -> Red
- D3: value LED -> Green
- R1: value R -> 39k
- R10: value R -> 5.1k
- R2: value R -> 100k
- R3: value R -> 15k
- R4: value R -> 470
- R5: value 4.7k -> 1k
- R6: value R -> 3k
- R7: value R -> 10k
- R8: value R -> 10M
- R9: value R -> 680k
Connections:
- net +BATT: now also M1.2; no longer M1.1
- net LED: now also D1.17 (PA15); no longer D1.7 (PA2)
- net Sound: now also D1.15 (PB4); no longer D1.9 (PA0)
- net Vibro: now also D1.16 (PB3); no longer D1.15 (PB4)
- net batLev: now also D1.6 (PA5); no longer D1.16 (PB3)
- net comLev: now also D1.7 (PA2); no longer D1.17 (PA15)
- net at Q2.3 (D): now also M1.1; no longer M1.2

Commit message: изменено:      kicad/bluz_v1/bluz_v1.kicad_pcb 	изменено:      kicad/bluz_v1/bluz_v1.kicad_sch
Parts:
- added C18: .1, Capacitor_SMD:C_0402_1005Metric, symbol Device:C
- added C20: 4.7u, Capacitor_SMD:C_0402_1005Metric, symbol Device:C
- R10: value 5.1k -> 75k
- R15: value 4.3M -> 5.1M
- R9: value 680k -> 10M
Connections:
- net B+: now also C20.1
- net GND: now also C18.1, C20.2
- net at D1.24 (RST), J2.1: now also C18.2
Other:
- moved on the sheet: D5, M1

Commit message: изменено:      Documents/BluZ.png 	изменено:      kicad/bluz_v1/bluz_v1.kicad_pcb 	изменено:      kicad/bluz_v1/bluz_v1.kicad_prl 	изменено:      kicad/bluz_v1/bluz_v1.kicad_sch 	изменено:      kicad/bluz_v1/fp-info-cache
Parts:
- added C21, C22: 10p, Capacitor_SMD:C_0402_1005Metric, symbol Device:C
- added Y2: NX1610-32.768, Crystal:Crystal_SMD_2012-2Pin_2.0x1.2mm, symbol Device:Crystal_Small
- L2: value 220uH -> 22uH
- Y1: value NX2016SA-32MHz -> NX1612SA-32MHz; footprint Crystal:Crystal_SMD_2016-4Pin_2.0x1.6mm -> My-library:NX1612SA
Connections:
- net AIn: now also D1.9 (PA0); no longer D1.8 (PA1)
- net GND: now also C21.2, C22.2
- net LED: now also D1.18 (PA14(swc)), J5.1; no longer D1.17 (PA15)
- net Sync: now also D1.17 (PA15); no longer D1.12 (PC15)
- net Vibro: now also D1.4 (PA6); no longer D1.16 (PB3)
- net comLev: now also D1.8 (PA1); no longer D1.7 (PA2)
- net at D1.13 (PC14): now also C21.1, Y2.2
- net swd: now reaches D1.19 (PA13(swd)), J4.1
- new net: C22.1, D1.12 (PC15), Y2.1
- no-connect marks 5 -> 4
Other:
- moved on the sheet: M1

Commit message: изменено:      kicad/bluz_v1/bluz_v1.kicad_pcb 	изменено:      kicad/bluz_v1/bluz_v1.kicad_prl 	изменено:      kicad/bluz_v1/bluz_v1.kicad_sch 	изменено:      kicad/bluz_v1/fp-info-cache
Parts:
- added J10, J9: Conn, lib:conn_mini, symbol My-Library:Conn
- BZ1: footprint MyLibrary:Buzzer55x55 -> My-library:Buzzer55x55
- C21, C22: footprint Capacitor_SMD:C_0402_1005Metric -> My-library:C_0201_0603Metric
- M1: footprint MyLibrary:VibroMotor -> My-library:VibroMotor
Connections:
- net GND: now also J10.1
- net TxD: now reaches D1.20 (PA12(rf_ant))
- net TxD: now also J9.1
- no-connect marks 4 -> 3

Commit message: новый файл:    Documents/BluZ-3D-Bot.png 	новый файл:    Documents/BluZ-3D-Top.png 	новый файл:    Documents/c_NX1610SE_e.pdf 	новый файл:    Documents/c_NX1612SA_e.pdf 	изменено:      README.md 	изменено:      kicad/bluz_v1/bluz_v1.kicad_pcb 	изменено:      kicad/bluz_v1/bluz_v1.kicad_sch 	изменено:      kicad/bluz_v1/fp-info-cache
Parts:
- Q1, Q2: footprint Package_TO_SOT_SMD:SOT-723 -> My-library:SOT-723
Changed lines of the file:
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@@
       (effects (font (size 1.27 1.27)) (justify left))
     )
-    (property "Footprint" "Package_TO_SOT_SMD:SOT-723" (id 2) (at 147.955 114.935 0)
+    (property "Footprint" "My-library:SOT-723" (id 2) (at 147.955 114.935 0)
       (effects (font (size 1.27 1.27)) hide)
     )
@@
       (effects (font (size 1.27 1.27)) (justify left))
     )
-    (property "Footprint" "Package_TO_SOT_SMD:SOT-723" (id 2) (at 164.465 114.935 0)
+    (property "Footprint" "My-library:SOT-723" (id 2) (at 164.465 114.935 0)
       (effects (font (size 1.27 1.27)) hide)
     )
@@
     )
     (path "/023c9820-1d2c-4bbf-b944-cb0d2cdd9333"
-      (reference "Q1") (unit 1) (value "RUM002N05") (footprint "Package_TO_SOT_SMD:SOT-723")
+      (reference "Q1") (unit 1) (value "RUM002N05") (footprint "My-library:SOT-723")
     )
     (path "/319576f9-2cb0-4f46-bd3c-2849efa10845"
-      (reference "Q2") (unit 1) (value "RUM002N05") (footprint "Package_TO_SOT_SMD:SOT-723")
+      (reference "Q2") (unit 1) (value "RUM002N05") (footprint "My-library:SOT-723")
     )
     (path "/0884e69a-0118-4e3d-a73e-60459bf2172a"

Commit message: изменено:      Documents/BluZ-3D-Bot.png 	изменено:      Documents/BluZ-3D-Top.png 	изменено:      Documents/BluZ.png 	изменено:      kicad/bluz_v1/bluz_v1.kicad_pcb 	изменено:      kicad/bluz_v1/bluz_v1.kicad_sch 	изменено:      kicad/bluz_v1/fp-info-cache
Parts:
- added C23: 10u, Capacitor_SMD:C_0402_1005Metric, symbol Device:C
- R1: value 39k -> 510k
- R2: value 100k -> 1M
- Y2: footprint Crystal:Crystal_SMD_2012-2Pin_2.0x1.2mm -> My-library:Crystal_SMD_2012-2Pin_2.0x1.2mm
Connections:
- net GND: now also R2.2, C23.2
- net LED: now also D1.7 (PA2); no longer D1.18 (PA14(swc)), J5.1
- net batLev: now also D1.8 (PA1); no longer D1.6 (PA5)
- net at C8.1, D1.5 (VDA), L1.2: now also C23.1
- removed net comLev: D1.8 (PA1), R2.2
- new net swc: D1.18 (PA14(swc)), J5.1

Commit message: изменено:      kicad/bluz_v1/bluz_v1.kicad_pcb 	изменено:      kicad/bluz_v1/bluz_v1.kicad_prl 	изменено:      kicad/bluz_v1/bluz_v1.kicad_sch
Connections:
- no-connect marks 3 -> 6
Other:
- moved on the sheet: D5, M1, U2

Commit message: изменено:      kicad/bluz_v1/bluz_v1.kicad_pcb 	изменено:      kicad/bluz_v1/bluz_v1.kicad_sch 	изменено:      kicad/bluz_v1/fp-info-cache
Parts:
- C12: value .1 -> 10n
- C16, C19: footprint Capacitor_SMD:C_0805_2012Metric -> Capacitor_SMD:C_1206_3216Metric
