File: kicad/bluz_v1/bluz_v1.kicad_sch (KiCad schematic)
At the start: 71 parts, among them J1 USB_B_Micro, J10 Conn, J11 Conn, J12 BTAnt, J2 Conn, J3 Conn, J4 Conn, J5 Conn, J6 Conn, J7 Conn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

Commit message: изменено:      kicad/bluz_v1/bluz_v1.kicad_sch 	изменено:      stm32cubeide/BluZ_v1/BluZ_v1.ioc 	изменено:      stm32cubeide/BluZ_v1/Core/Inc/app_conf.h 	изменено:      stm32cubeide/BluZ_v1/Core/Inc/main.h 	изменено:      stm32cubeide/BluZ_v1/Core/Src/main.c 	изменено:      stm32cubeide/BluZ_v1/Core/Src/stm32wbaxx_it.c 	изменено:      stm32cubeide/BluZ_v1/Release/BluZ_v1.hex 	изменено:      stm32cubeide/BluZ_v1/Release/BluZ_v1.list 	изменено:      stm32cubeide/BluZ_v1/Release/BluZ_v1.map 	изменено:      stm32cubeide/BluZ_v1/Release/Core/Src/app_entry.d 	изменено:      stm32cubeide/BluZ_v1/Release/STM32_WPAN/Target/linklayer_plat.d
Parts:
- C1, C11, C14, C2, C20, C24, C3, C5, C6: value 4.7u -> 22u
- C10, C13, C15, C23, C4, C8: value 10u -> 22u
- C18: value .1 -> 10n
Other:
- note added: "Токи периферии: MCP1700 - 1.6uA LTC1662C - 1,5uA * 2 AP3015 - 52uA (run) TLV3201 - 40uA CompRef - 0.3uA BatLev - 2.7uA MCP73831 - 2uA ------------- Total: 101.6uA Real: 90uA"
- note removed: "Токи периферии: MCP1700 - 1.6uA LTC1662C - 1,5uA * 2 AP3015 - 52uA (run) TLV3201 - 40uA CompRef - 0.3uA BatLev - 2.7uA MCP73831 - 2uA ------------- Total: 101.6uA Real: 89.9uA"
Changed lines of the file:
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@@
     )
   )
-  (text "Токи периферии:\nMCP1700 - 1.6uA\nLTC1662C - 1,5uA * 2\nAP3015 - 52uA (run)\nTLV3201 - 40uA\nCompRef - 0.3uA\nBatLev - 2.7uA\nMCP73831 - 2uA\n-------------\nTotal: 101.6uA\nReal: 89.9uA\n"
+  (text "Токи периферии:\nMCP1700 - 1.6uA\nLTC1662C - 1,5uA * 2\nAP3015 - 52uA (run)\nTLV3201 - 40uA\nCompRef - 0.3uA\nBatLev - 2.7uA\nMCP73831 - 2uA\n-------------\nTotal: 101.6uA\nReal: 90uA\n"
     (at 217.17 39.37 0)
     (effects (font (size 1.27 1.27)) (justify left bottom))
@@
       (effects (font (size 1.27 1.27)) hide)
     )
-    (property "Value" "4.7u" (id 1) (at 159.385 95.885 0))
+    (property "Value" "22u" (id 1) (at 159.385 95.885 0))
     (property "Footprint" "Capacitor_SMD:C_0402_1005Metric" (id 2) (at 155.2448 94.615 0)
       (effects (font (size 1.27 1.27)) hide)
@@
       (effects (font (size 1.27 1.27)) (justify left) hide)
     )
-    (property "Value" "4.7u" (id 1) (at 69.215 50.8 0)
+    (property "Value" "22u" (id 1) (at 69.215 50.8 0)
       (effects (font (size 1.27 1.27)) (justify left))
     )
@@
       (effects (font (size 1.27 1.27)) (justify left) hide)
     )
-    (property "Value" "10u" (id 1) (at 131.445 40.005 0)
+    (property "Value" "22u" (id 1) (at 131.445 40.005 0)
       (effects (font (size 1.27 1.27)) (justify left))
     )
@@
   )
   (symbol (lib_id "Device:R") (at 99.695 23.495 90) (unit 1)
-    (in_bom yes) (on_board yes) (fields_autoplaced)
+    (in_bom yes) (on_board yes)
     (property "Reference" "R4" (id 0) (at 99.695 18.7792 90)
       (effects (font (size 1.27 1.27)) hide)
     )
-    (property "Value" "220" (id 1) (at 99.695 19.685 90))
+    (property "Value" "220" (id 1) (at 99.695 20.955 90))
     (property "Footprint" "Resistor_SMD:R_0402_1005Metric" (id 2) (at 99.695 25.273 90)
       (effects (font (size 1.27 1.27)) hide)
@@
       (effects (font (size 1.27 1.27)) hide)
     )
-    (property "Value" "10u" (id 1) (at 97.155 46.99 90))
+    (property "Value" "22u" (id 1) (at 97.155 46.99 90))
     (property "Footprint" "Capacitor_SMD:C_0402_1005Metric" (id 2) (at 104.14 47.2948 0)
       (effects (font (size 1.27 1.27)) hide)
@@
       (effects (font (size 1.27 1.27)) (justify left) hide)
     )
-    (property "Value" "4.7u" (id 1) (at 120.015 53.975 0)
+    (property "Value" "22u" (id 1) (at 120.015 53.975 0)
       (effects (font (size 1.27 1.27)) (justify left))
     )
@@
       (effects (font (size 1.27 1.27)) (justify left) hide)
     )
-    (property "Value" "4.7u" (id 1) (at 110.49 35.56 0)
+    (property "Value" "22u" (id 1) (at 110.49 35.56 0)
       (effects (font (size 1.27 1.27)) (justify left))
     )
@@
       (effects (font (size 1.27 1.27)) (justify left) hide)
     )
-    (property "Value" "4.7u" (id 1) (at 64.135 50.8 0)
+    (property "Value" "22u" (id 1) (at 64.135 50.8 0)
       (effects (font (size 1.27 1.27)) (justify left))
     )
@@
       (effects (font (size 1.27 1.27)) (justify left) hide)
     )
-    (property "Value" "10u" (id 1) (at 67.31 38.1 0)
+    (property "Value" "22u" (id 1) (at 67.31 38.1 0)
       (effects (font (size 1.27 1.27)) (justify left))
     )
@@
       (effects (font (size 1.27 1.27)) (justify left) hide)
     )
-    (property "Value" "4.7u" (id 1) (at 74.295 50.8 0)
+    (property "Value" "22u" (id 1) (at 74.295 50.8 0)
       (effects (font (size 1.27 1.27)) (justify left))
     )
@@
       (effects (font (size 1.27 1.27)) (justify right) hide)
     )
-    (property "Value" "10u" (id 1) (at 140.97 35.56 0)
+    (property "Value" "22u" (id 1) (at 140.97 35.56 0)
       (effects (font (size 1.27 1.27)) (justify right))
     )
@@
       (effects (font (size 1.27 1.27)) hide)
     )
-    (property "Value" "10u" (id 1) (at 100.965 57.15 90))
+    (property "Value" "22u" (id 1) (at 100.965 57.15 90))
     (property "Footprint" "Capacitor_SMD:C_0402_1005Metric" (id 2) (at 104.14 52.3748 0)
       (effects (font (size 1.27 1.27)) hide)
@@
       (effects (font (size 1.27 1.27)) (justify left) hide)
     )
-    (property "Value" "10u" (id 1) (at 118.745 40.005 0)
+    (property "Value" "22u" (id 1) (at 118.745 40.005 0)
       (effects (font (size 1.27 1.27)) (justify left))
     )
@@
       (effects (font (size 1.27 1.27)) hide)
     )
-    (property "Value" "4.7u" (id 1) (at 172.72 72.39 90))
+    (property "Value" "22u" (id 1) (at 172.72 72.39 90))
     (property "Footprint" "Capacitor_SMD:C_0402_1005Metric" (id 2) (at 176.53 67.6148 0)
       (effects (font (size 1.27 1.27)) hide)
@@
       (effects (font (size 1.27 1.27)) (justify left) hide)
     )
-    (property "Value" "4.7u" (id 1) (at 79.375 50.8 0)
+    (property "Value" "22u" (id 1) (at 79.375 50.8 0)
       (effects (font (size 1.27 1.27)) (justify left))
     )
@@
       (effects (font (size 1.27 1.27)) (justify left) hide)
     )
-    (property "Value" "4.7u" (id 1) (at 59.055 50.8 0)
+    (property "Value" "22u" (id 1) (at 59.055 50.8 0)
       (effects (font (size 1.27 1.27)) (justify left))
     )
@@
       (effects (font (size 1.27 1.27)) hide)
     )
-    (property "Value" ".1" (id 1) (at 64.135 69.215 0))
+    (property "Value" "10n" (id 1) (at 64.135 69.215 0))
     (property "Footprint" "Capacitor_SMD:C_0402_1005Metric" (id 2) (at 65.0748 62.865 0)
       (effects (font (size 1.27 1.27)) hide)
@@
     )
     (path "/e8a689ec-473b-41cb-80a7-1d113ee6c137"
-      (reference "C1") (unit 1) (value "4.7u") (footprint "Capacitor_SMD:C_0402_1005Metric")
+      (reference "C1") (unit 1) (value "22u") (footprint "Capacitor_SMD:C_0402_1005Metric")
     )
     (path "/6fd9cfa6-88d8-4773-b9f2-131d75673dd7"
-      (reference "C2") (unit 1) (value "4.7u") (footprint "Capacitor_SMD:C_0402_1005Metric")
+      (reference "C2") (unit 1) (value "22u") (footprint "Capacitor_SMD:C_0402_1005Metric")
     )
     (path "/22fba23d-97b7-4b53-8ff8-23b0a511477e"
-      (reference "C3") (unit 1) (value "4.7u") (footprint "Capacitor_SMD:C_0402_1005Metric")
+      (reference "C3") (unit 1) (value "22u") (footprint "Capacitor_SMD:C_0402_1005Metric")
     )
     (path "/70383fc7-eca8-4756-8c22-2aa2624acf07"
-      (reference "C4") (unit 1) (value "10u") (footprint "Capacitor_SMD:C_0402_1005Metric")
+      (reference "C4") (unit 1) (value "22u") (footprint "Capacitor_SMD:C_0402_1005Metric")
     )
     (path "/8c25cba8-5ac8-437d-a59e-8abcf99ef9a2"
-      (reference "C5") (unit 1) (value "4.7u") (footprint "Capacitor_SMD:C_0402_1005Metric")
+      (reference "C5") (unit 1) (value "22u") (footprint "Capacitor_SMD:C_0402_1005Metric")
     )
     (path "/ce4b8343-c432-43f5-be1c-455dfe61e55a"
-      (reference "C6") (unit 1) (value "4.7u") (footprint "Capacitor_SMD:C_0402_1005Metric")
+      (reference "C6") (unit 1) (value "22u") (footprint "Capacitor_SMD:C_0402_1005Metric")
     )
     (path "/cda4b512-0c1b-492b-8015-89931185c3a4"
@@
     )
     (path "/9582b2c0-dd8d-4f39-be71-175493c3a453"
-      (reference "C8") (unit 1) (value "10u") (footprint "Capacitor_SMD:C_0402_1005Metric")
+      (reference "C8") (unit 1) (value "22u") (footprint "Capacitor_SMD:C_0402_1005Metric")
     )
     (path "/386fe074-b839-4ef8-9e75-b78b50bc29fe"
@@
     )
     (path "/b484d6c5-39be-4be9-a936-ddec27e5986f"
-      (reference "C10") (unit 1) (value "10u") (footprint "Capacitor_SMD:C_0402_1005Metric")
+      (reference "C10") (unit 1) (value "22u") (footprint "Capacitor_SMD:C_0402_1005Metric")
     )
     (path "/3f1a12d4-3545-4b60-949b-d28c5a4b97fb"
-      (reference "C11") (unit 1) (value "4.7u") (footprint "Capacitor_SMD:C_0402_1005Metric")
+      (reference "C11") (unit 1) (value "22u") (footprint "Capacitor_SMD:C_0402_1005Metric")
     )
     (path "/95b828e2-2230-4d8c-b384-f5b115a71403"
@@
     )
     (path "/3795737e-81b8-472d-94be-3f8dcbb66065"
-      (reference "C13") (unit 1) (value "10u") (footprint "Capacitor_SMD:C_0402_1005Metric")
+      (reference "C13") (unit 1) (value "22u") (footprint "Capacitor_SMD:C_0402_1005Metric")
     )
     (path "/bd5cecec-cebb-4331-9968-eb56d44e302e"
-      (reference "C14") (unit 1) (value "4.7u") (footprint "Capacitor_SMD:C_0402_1005Metric")
+      (reference "C14") (unit 1) (value "22u") (footprint "Capacitor_SMD:C_0402_1005Metric")
     )
     (path "/8f3c1956-d483-4ba9-91db-59fe3f3512b6"
-      (reference "C15") (unit 1) (value "10u") (footprint "Capacitor_SMD:C_0402_1005Metric")
+      (reference "C15") (unit 1) (value "22u") (footprint "Capacitor_SMD:C_0402_1005Metric")
     )
     (path "/16bbbb75-6154-486b-84f6-0c1483bc5f51"
@@
     )
     (path "/f2d24064-1ea8-4940-bbc5-ff6713d4e4b5"
-      (reference "C18") (unit 1) (value ".1") (footprint "Capacitor_SMD:C_0402_1005Metric")
+      (reference "C18") (unit 1) (value "10n") (footprint "Capacitor_SMD:C_0402_1005Metric")
     )
     (path "/134867a7-9699-4483-af4a-0e90ac8f8405"
@@
     )
     (path "/6916de32-6e66-4bee-aa98-6c0b14bb45bd"
-      (reference "C20") (unit 1) (value "4.7u") (footprint "Capacitor_SMD:C_0402_1005Metric")
+      (reference "C20") (unit 1) (value "22u") (footprint "Capacitor_SMD:C_0402_1005Metric")
     )
     (path "/2e49414d-2639-4544-8e9e-3340fed11837"
@@
     )
     (path "/3ac87482-ffff-4971-8823-9ea94a9136ed"
-      (reference "C23") (unit 1) (value "10u") (footprint "Capacitor_SMD:C_0402_1005Metric")
+      (reference "C23") (unit 1) (value "22u") (footprint "Capacitor_SMD:C_0402_1005Metric")
     )
     (path "/0118fc95-6142-48f8-a925-bca7546c2bd0"
-      (reference "C24") (unit 1) (value "4.7u") (footprint "Capacitor_SMD:C_0402_1005Metric")
+      (reference "C24") (unit 1) (value "22u") (footprint "Capacitor_SMD:C_0402_1005Metric")
     )
     (path "/0b18ea72-3ce5-4bf2-8abb-f59f2457f733"

Commit message: изменено:      kicad/bluz_v1/bluz_v1.kicad_pcb 	изменено:      kicad/bluz_v1/bluz_v1.kicad_sch
Parts:
- Y2: value NX1610-32.768 -> NX2010SA-32.768
Changed lines of the file:
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@@
       (effects (font (size 1.27 1.27)) hide)
     )
-    (property "Value" "NX1610-32.768" (id 1) (at 115.57 80.645 0))
+    (property "Value" "NX2010SA-32.768" (id 1) (at 115.57 80.645 0))
     (property "Footprint" "My-library:Crystal_SMD_2012-2Pin_2.0x1.2mm" (id 2) (at 113.665 86.36 0)
       (effects (font (size 1.27 1.27)) hide)
@@
     )
     (path "/5f4215d5-5c6c-4709-b145-abb58fc32108"
-      (reference "Y2") (unit 1) (value "NX1610-32.768") (footprint "My-library:Crystal_SMD_2012-2Pin_2.0x1.2mm")
-    )
-  )
+      (reference "Y2") (unit 1) (value "NX2010SA-32.768") (footprint "My-library:Crystal_SMD_2012-2Pin_2.0x1.2mm")
+    )
+  )

Commit message: изменено:      kicad/bluz_v1/bluz_v1.kicad_pcb 	изменено:      kicad/bluz_v1/bluz_v1.kicad_sch
Parts:
- Y2: value NX2010SA-32.768 -> NX2012SA-32.768
Changed lines of the file:
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@@
       (effects (font (size 1.27 1.27)) hide)
     )
-    (property "Value" "NX2010SA-32.768" (id 1) (at 115.57 80.645 0))
+    (property "Value" "NX2012SA-32.768" (id 1) (at 115.57 80.645 0))
     (property "Footprint" "My-library:Crystal_SMD_2012-2Pin_2.0x1.2mm" (id 2) (at 113.665 86.36 0)
       (effects (font (size 1.27 1.27)) hide)
@@
     )
     (path "/5f4215d5-5c6c-4709-b145-abb58fc32108"
-      (reference "Y2") (unit 1) (value "NX2010SA-32.768") (footprint "My-library:Crystal_SMD_2012-2Pin_2.0x1.2mm")
-    )
-  )
+      (reference "Y2") (unit 1) (value "NX2012SA-32.768") (footprint "My-library:Crystal_SMD_2012-2Pin_2.0x1.2mm")
+    )
+  )
