File: kicad/bluz_Macropixel/bluz_Macropixel.kicad_pcb (KiCad board)
At the start: 2 copper layers, 50.3 x 19.8 mm, 67 parts, among them J1 USB_B_Micro, J10 Conn, J11 Conn_01x06_Female, J12 BTAnt, J13 Conn_01x06_Female, J2 Conn, J3 Conn, J4 Conn, J5 Conn, J6 Conn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

Commit message: изменено:      kicad/bluz_Macropixel/bluz_Macropixel.kicad_pcb 	изменено:      kicad/bluz_Macropixel/bluz_Macropixel.kicad_prl 	изменено:      kicad/bluz_Macropixel/bluz_Macropixel.kicad_pro 	изменено:      kicad/bluz_Macropixel/bluz_Macropixel.kicad_sch 	изменено:      kicad/bluz_Macropixel/fp-info-cache
Parts:
- removed J3: Conn, lib:conn_mini
- moved R14 13.2 mm to (83.1, 38.1)
- moved R9 2.00 mm to (80.5, 45.6), turned to 0 degrees
- moved J13 1.88 mm to (87.6, 38.4)
- moved R5 1.23 mm to (81.4, 45.0)
- moved C17 0.72 mm to (73.8, 38.0)
- moved D6 0.33 mm to (72.4, 39.4)
- moved C11 0.27 mm to (82.4, 43.9)
- moved D3 0.24 mm to (80.4, 43.9)
Routing:
- net +SiPM: track 20.0 -> 4.38 mm
- net Net-(D5-K): track 7.26 -> 19.1 mm
- net GND: track 125.5 -> 113.8 mm
- net SCL: track 22.5 -> 20.7 mm
- net +2V8: track 40.6 -> 42.3 mm
- net SDA: track 22.3 -> 20.7 mm
- net -SiPM: track 20.1 -> 21.5 mm
- net batLev: track 19.0 -> 19.7 mm
- net Net-(D1-VDDHPA): track 1.65 -> 2.27 mm
Other:
- outline, holes or cut-outs redrawn

Commit message: изменено:      kicad/bluz_Macropixel/bluz_Macropixel.kicad_pcb 	изменено:      kicad/bluz_Macropixel/bluz_Macropixel.kicad_pro 	изменено:      kicad/bluz_Macropixel/bluz_Macropixel.kicad_sch
Parts:
- removed J9: Conn, lib:conn_mini
- C11: moved to F.Cu
- D5: value BAT46JFILM -> BAS516; footprint Diode_SMD:D_SOD-323 -> Diode_SMD:D_SOD-523
- moved C11 4.15 mm to (80.0, 40.5)
- moved C16 1.42 mm to (69.9, 39.6)
- moved D5 0.28 mm to (67.7, 41.5)
- moved L2 0.14 mm to (64.3, 41.8)
Connections:
- D1 pad 20: /TxD -> unconnected-(D1-PA12-Pad20)
Routing:
- net /TxD: track 9.75 -> 0.00 mm
- net GND: track 113.8 -> 115.9 mm
- net Sync: track 19.8 -> 18.0 mm
- net Net-(D5-K): track 19.1 -> 17.7 mm
- net HVAdj: track 20.8 -> 20.1 mm
- net batLev: track 19.7 -> 19.0 mm
