File: kicad/bluz_Macropixel/bluz_Macropixel.kicad_sch (KiCad schematic)
At the start: 67 parts, among them J1 USB_B_Micro, J10 Conn, J11 Conn_01x06_Female, J12 BTAnt, J13 Conn_01x06_Female, J2 Conn, J3 Conn, J4 Conn, J5 Conn, J6 Conn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

Commit message: изменено:      kicad/bluz_Macropixel/bluz_Macropixel.kicad_pcb 	изменено:      kicad/bluz_Macropixel/bluz_Macropixel.kicad_prl 	изменено:      kicad/bluz_Macropixel/bluz_Macropixel.kicad_pro 	изменено:      kicad/bluz_Macropixel/bluz_Macropixel.kicad_sch 	изменено:      kicad/bluz_Macropixel/fp-info-cache
Parts:
- removed J3: Conn, lib:conn_mini, symbol My-Library:Conn

Commit message: изменено:      kicad/bluz_Macropixel/bluz_Macropixel.kicad_pcb 	изменено:      kicad/bluz_Macropixel/bluz_Macropixel.kicad_pro 	изменено:      kicad/bluz_Macropixel/bluz_Macropixel.kicad_sch
Parts:
- removed J9: Conn, lib:conn_mini, symbol My-Library:Conn
- D5: value BAT46JFILM -> BAS516; footprint Diode_SMD:D_SOD-323 -> Diode_SMD:D_SOD-523
Connections:
- net TxD: no longer names the net of D1.20 (PA12)
- no-connect marks 6 -> 7
