File: kicad/bluz_v1_typec/bluz_v1.kicad_sch (KiCad schematic)
At the start: 72 parts, among them J10 Conn, J11 Conn, J12 BTAnt, J2 Conn, J3 Conn, J4 Conn, J5 Conn, J6 Conn, J7 Conn, J8 Conn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

Commit message: изменено:      Android/BluZ_LPM/BluZ/src/main/java/ru/starline/bluz/NumberFragment.kt 	изменено:      Android/BluZ_LPM/BluZ/src/main/java/ru/starline/bluz/drawSpecter.kt 	изменено:      Android/BluZ_LPM/BluZ/src/main/java/ru/starline/bluz/globalObj.kt 	изменено:      Android/BluZ_LPM/BluZ/src/main/res/layout/setup_layout.xml 	изменено:      kicad/bluz_v1_typec/bluz_v1.kicad_sch 	изменено:      kicad/bluz_v2_typec/bluz_v1.kicad_pcb 	изменено:      kicad/bluz_v2_typec/bluz_v1.kicad_pro 	изменено:      kicad/bluz_v2_typec/fp-info-cache 	изменено:      stm32cubeide/BluZ_LPM/BluZ_LPM.ioc 	изменено:      stm32cubeide/BluZ_LPM/Core/Src/main.c 	изменено:      stm32cubeide/BluZ_LPM/Release/BluZ_LPM.elf
Changed lines of the file:
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@@
 		(dnp no)
 		(property "Reference" "R10"
-			(at 172.593 103.3053 0)
+			(at 165.608 103.886 0)
 			(effects
 				(font
@@
 				)
 				(justify left)
-				(hide yes)
 			)
 		)
@@
 		(dnp no)
 		(property "Reference" "R6"
-			(at 164.338 103.3053 0)
+			(at 158.75 103.632 0)
 			(effects
 				(font
@@
 				)
 				(justify left)
-				(hide yes)
 			)
 		)
@@
 		(on_board yes)
 		(dnp no)
-		(fields_autoplaced yes)
 		(property "Reference" "R7"
-			(at 166.37 94.3442 90)
+			(at 167.64 95.25 90)
 			(effects
 				(font
 					(size 1.27 1.27)
 				)
-				(hide yes)
 			)
 		)
 		(property "Value" "10k"
-			(at 166.37 96.8812 90)
+			(at 167.894 97.028 90)
 			(effects
 				(font
@@
 		(dnp no)
 		(property "Reference" "C12"
-			(at 177.546 103.3053 0)
+			(at 179.324 104.648 0)
 			(effects
 				(font
@@
 				)
 				(justify left)
-				(hide yes)
 			)
 		)
 		(property "Value" "10n"
-			(at 175.26 106.68 0)
+			(at 179.578 106.68 0)
 			(effects
 				(font
@@
 		(dnp no)
 		(property "Reference" "R9"
-			(at 172.593 89.3353 0)
+			(at 172.72 88.138 0)
 			(effects
 				(font
@@
 				)
 				(justify left)
-				(hide yes)
 			)
 		)
@@
 		(dnp no)
 		(property "Reference" "C14"
-			(at 182.88 80.5012 90)
+			(at 183.134 89.916 90)
 			(effects
 				(font
 					(size 1.27 1.27)
 				)
-				(hide yes)
 			)
 		)
 		(property "Value" "22u"
-			(at 182.88 90.17 90)
+			(at 182.88 91.948 90)
 			(effects
 				(font
@@
 		(dnp no)
 		(property "Reference" "R8"
-			(at 169.418 89.3353 0)
+			(at 163.068 89.662 0)
 			(effects
 				(font
@@
 				)
 				(justify left)
-				(hide yes)
 			)
 		)
 		(property "Value" "10M"
-			(at 161.925 90.17 0)
+			(at 162.052 91.694 0)
 			(effects
 				(font
