File: kicad/bluz_v1_typec/bluz_v1.kicad_pcb (KiCad board)
At the start: 2 copper layers, 24.9 x 14.9 mm, 72 parts, among them J10 Conn, J11 Conn, J12 BTAnt, J2 Conn, J3 Conn, J4 Conn, J5 Conn, J6 Conn, J7 Conn, J8 Conn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

Commit message: изменено:      kicad/bluz_v1_typec/bluz_v1.kicad_pcb 	изменено:      kicad/bluz_v1_typec/bluz_v1.kicad_sch 	изменено:      kicad/bluz_v1_typec/bom/ibom.html
Parts:
- BZ1: value Buzzer -> MLT-5020
- M1: value VibroMotor -> Z3OC1T8219731
Changed lines of the file:
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@@
 			)
 		)
-		(property "Datasheet" ""
+		(property "Datasheet" "~"
 			(at 0 0 270)
 			(layer "F.Fab")
@@
 			)
 		)
-		(property "Datasheet" ""
+		(property "Datasheet" "~"
 			(at 0 0 90)
 			(layer "F.Fab")
@@
 			)
 		)
-		(property "Datasheet" ""
+		(property "Datasheet" "~"
 			(at 0 0 0)
 			(layer "F.Fab")
@@
 			)
 		)
-		(property "Datasheet" ""
+		(property "Datasheet" "~"
 			(at 0 0 180)
 			(layer "F.Fab")
@@
 			)
 		)
-		(property "Datasheet" ""
+		(property "Datasheet" "~"
 			(at 0 0 180)
 			(layer "B.Fab")
@@
 			)
 		)
-		(property "Datasheet" ""
+		(property "Datasheet" "~"
 			(at 0 0 270)
 			(layer "F.Fab")
@@
 			)
 		)
-		(property "Value" "VibroMotor"
+		(property "Value" "Z3OC1T8219731"
 			(at -5.8928 -4.7244 180)
 			(unlocked yes)
@@
 			)
 		)
-		(property "Datasheet" ""
+		(property "Datasheet" "~"
 			(at 0 0 270)
 			(layer "F.Fab")
@@
 			)
 		)
-		(property "Datasheet" ""
+		(property "Datasheet" "~"
 			(at 0 0 180)
 			(layer "F.Fab")
@@
 			)
 		)
-		(property "Datasheet" ""
+		(property "Datasheet" "~"
 			(at 0 0 270)
 			(layer "F.Fab")
@@
 			)
 		)
-		(property "Datasheet" ""
+		(property "Datasheet" "~"
 			(at 0 0 180)
 			(layer "F.Fab")
@@
 			)
 		)
-		(property "Datasheet" ""
+		(property "Datasheet" "~"
 			(at 0 0 270)
 			(layer "F.Fab")
@@
 			)
 		)
-		(property "Value" "Buzzer"
+		(property "Value" "MLT-5020"
 			(at 0.19 4.72 90)
 			(unlocked yes)
@@
 			)
 		)
-		(property "Datasheet" ""
+		(property "Datasheet" "~"
 			(at 0 0 90)
 			(layer "B.Fab")
@@
 			)
 		)
-		(property "Datasheet" ""
+		(property "Datasheet" "~"
 			(at 0 0 0)
 			(layer "F.Fab")
@@
 			)
 		)
-		(property "Datasheet" ""
+		(property "Datasheet" "~"
 			(at 0 0 90)
 			(layer "F.Fab")
@@
 			)
 		)
-		(property "Datasheet" ""
+		(property "Datasheet" "~"
 			(at 0 0 270)
 			(layer "F.Fab")
@@
 			)
 		)
-		(property "Datasheet" ""
+		(property "Datasheet" "~"
 			(at 0 0 0)
 			(layer "F.Fab")
@@
 			)
 		)
-		(property "Datasheet" ""
+		(property "Datasheet" "~"
 			(at 0 0 90)
 			(layer "B.Fab")
@@
 			)
 		)
-		(property "Datasheet" ""
+		(property "Datasheet" "~"
 			(at 0 0 90)
 			(layer "F.Fab")
@@
 			)
 		)
-		(property "Datasheet" ""
+		(property "Datasheet" "~"
 			(at 0 0 90)
 			(layer "B.Fab")
@@
 			)
 		)
-		(property "Datasheet" ""
+		(property "Datasheet" "~"
 			(at 0 0 0)
 			(layer "B.Fab")
@@
 			)
 		)
-		(property "Datasheet" ""
+		(property "Datasheet" "~"
 			(at 0 0 90)
 			(layer "F.Fab")
@@
 			)
 		)
-		(property "Datasheet" ""
+		(property "Datasheet" "~"
 			(at 0 0 0)
 			(layer "F.Fab")
@@
 			)
 		)
-		(property "Datasheet" ""
+		(property "Datasheet" "~"
 			(at 0 0 0)
 			(layer "F.Fab")
@@
 			)
 		)
-		(property "Datasheet" ""
+		(property "Datasheet" "~"
 			(at 0 0 90)
 			(layer "F.Fab")
@@
 			)
 		)
-		(property "Datasheet" ""
+		(property "Datasheet" "~"
 			(at 0 0 180)
 			(layer "F.Fab")
@@
 			)
 		)
-		(property "Datasheet" ""
+		(property "Datasheet" "~"
 			(at 0 0 90)
 			(layer "F.Fab")
@@
 			)
 		)
-		(property "Datasheet" ""
+		(property "Datasheet" "~"
 			(at 0 0 270)
 			(layer "F.Fab")
@@
 			)
 		)
-		(property "Datasheet" ""
+		(property "Datasheet" "~"
 			(at 0 0 0)
 			(layer "F.Fab")
@@
 			)
 		)
-		(property "Datasheet" ""
+		(property "Datasheet" "~"
 			(at 0 0 270)
 			(layer "F.Fab")
@@
 			)
 		)
-		(property "Datasheet" ""
+		(property "Datasheet" "~"
 			(at 0 0 270)
 			(layer "F.Fab")
@@
 			)
 		)
-		(property "Datasheet" ""
+		(property "Datasheet" "~"
 			(at 0 0 270)
 			(layer "F.Fab")
@@
 			)
 		)
-		(property "Datasheet" ""
+		(property "Datasheet" "~"
 			(at 0 0 270)
 			(layer "F.Fab")
@@
 			)
 		)
-		(property "Datasheet" ""
+		(property "Datasheet" "~"
 			(at 0 0 180)
 			(layer "F.Fab")
@@
 			)
 		)
-		(property "Datasheet" ""
+		(property "Datasheet" "~"
 			(at 0 0 180)
 			(layer "F.Fab")
@@
 			)
 		)
-		(property "Datasheet" ""
+		(property "Datasheet" "~"
 			(at 0 0 90)
 			(layer "F.Fab")
@@
 			)
 		)
-		(property "Datasheet" ""
+		(property "Datasheet" "~"
 			(at 0 0 180)
 			(layer "F.Fab")
@@
 			)
 		)
-		(property "Datasheet" ""
+		(property "Datasheet" "~"
 			(at 0 0 0)
 			(layer "B.Fab")
@@
 			)
 		)
-		(property "Datasheet" ""
+		(property "Datasheet" "~"
 			(at 0 0 180)
 			(layer "F.Fab")
@@
 			)
 		)
-		(property "Datasheet" ""
+		(property "Datasheet" "~"
 			(at 0 0 90)
 			(layer "F.Fab")
@@
 			)
 		)
-		(property "Datasheet" ""
+		(property "Datasheet" "~"
 			(at 0 0 180)
 			(layer "B.Fab")
@@
 			)
 		)
-		(property "Datasheet" ""
+		(property "Datasheet" "~"
 			(at 0 0 90)
 			(layer "F.Fab")
@@
 			)
 		)
-		(property "Datasheet" ""
+		(property "Datasheet" "~"
 			(at 0 0 180)
 			(layer "F.Fab")
@@
 			)
 		)
-		(property "Datasheet" ""
+		(property "Datasheet" "~"
 			(at 0 0 180)
 			(layer "F.Fab")
@@
 			)
 		)
-		(property "Datasheet" ""
+		(property "Datasheet" "~"
 			(at 0 0 0)
 			(layer "F.Fab")
@@
 			)
 		)
-		(property "Datasheet" ""
+		(property "Datasheet" "~"
 			(at 0 0 0)
 			(layer "B.Fab")
@@
 			)
 		)
-		(property "Datasheet" ""
+		(property "Datasheet" "~"
 			(at 0 0 180)
 			(layer "F.Fab")
@@
 			)
 		)
-		(property "Datasheet" ""
+		(property "Datasheet" "~"
 			(at 0 0 180)
 			(layer "F.Fab")
@@
 			)
 		)
-		(property "Datasheet" ""
+		(property "Datasheet" "~"
 			(at 0 0 90)
 			(layer "F.Fab")
@@
 			)
 		)
-		(property "Datasheet" ""
+		(property "Datasheet" "~"
 			(at 0 0 180)
 			(layer "F.Fab")
@@
 			)
 		)
-		(property "Datasheet" ""
+		(property "Datasheet" "~"
 			(at 0 0 0)
 			(layer "F.Fab")
@@
 			)
 		)
-		(property "Datasheet" ""
+		(property "Datasheet" "~"
 			(at 0 0 180)
 			(layer "F.Fab")
@@
 			)
 		)
-		(property "Datasheet" ""
+		(property "Datasheet" "~"
 			(at 0 0 90)
 			(layer "F.Fab")
@@
 			)
 		)
-		(property "Datasheet" ""
+		(property "Datasheet" "~"
 			(at 0 0 90)
 			(layer "F.Fab")
@@
 			)
 		)
-		(property "Datasheet" ""
+		(property "Datasheet" "~"
 			(at 0 0 180)
 			(layer "F.Fab")
@@
 			)
 		)
-		(property "Datasheet" ""
+		(property "Datasheet" "~"
 			(at 0 0 0)
 			(layer "F.Fab")

Commit message: удалено:       kicad/bluz_v1_typec/bluz_v1-backups/bluz_v1-2025-08-04_173346.zip 	изменено:      kicad/bluz_v1_typec/bluz_v1.kicad_pcb 	изменено:      kicad/bluz_v1_typec/bluz_v1.kicad_sch 	изменено:      kicad/bluz_v1_typec/bom/ibom.html
Parts:
- D5: value BAS16 -> BAS16J
Changed lines of the file:
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@@
 			)
 		)
-		(property "Value" "BAS16"
+		(property "Value" "BAS16J"
 			(at 0.1 1.9 90)
 			(layer "F.Fab")

Commit message: изменено:      Android/BluZ_LPM/BluZ/src/main/java/ru/starline/bluz/NumberFragment.kt 	изменено:      kicad/bluz_v1_typec/bluz_v1.kicad_pcb 	изменено:      stm32cubeide/BluZ_LPM/BluZ_LPM_v1.ioc 	изменено:      stm32cubeide/BluZ_LPM/Core/Inc/app_conf.h 	изменено:      stm32cubeide/BluZ_LPM/Core/Src/main.c 	изменено:      stm32cubeide/BluZ_LPM/Release/BluZ_LPM_v1.elf 	изменено:      stm32cubeide/BluZ_LPM/STM32_WPAN/App/app_ble.c 	изменено:      stm32cubeide/BluZ_archive/.cproject 	изменено:      stm32cubeide/BluZ_archive/.mxproject 	изменено:      stm32cubeide/BluZ_archive/.settings/language.settings.xml 	изменено:      stm32cubeide/BluZ_archive/BluZ_v1.ioc 	изменено:      stm32cubeide/BluZ_archive/Core/Inc/app_common.h 	изменено:      stm32cubeide/BluZ_archive/Core/Inc/app_conf.h 	изменено:      stm32cubeide/BluZ_archive/Core/Inc/main.h 	изменено:      stm32cubeide/BluZ_archive/Core/Inc/stm32wbaxx_hal_conf.h 	изменено:      stm32cubeide/BluZ_archive/Core/Inc/stm32wbaxx_it.h 	изменено:      stm32cubeide/BluZ_archive/Core/Inc/utilities_conf.h 	изменено:      stm32cubeide/BluZ_archive/Core/Src/app_entry.c 	изменено:      stm32cubeide/BluZ_archive/Core/Src/main.c 	изменено:      stm32cubeide/BluZ_archive/Core/Src/stm32wbaxx_hal_msp.c 	изменено:      stm32cubeide/BluZ_archive/Core/Src/stm32wbaxx_it.c 	изменено:      stm32cubeide/BluZ_archive/Drivers/CMSIS/Device/ST/STM32WBAxx/Include/stm32wba54xx.h 	изменено:      stm32cubeide/BluZ_archive/Drivers/CMSIS/Device/ST/STM32WBAxx/Include/stm32wbaxx.h 	изменено:      stm32cubeide/BluZ_archive/Drivers/CMSIS/Device/ST/STM32WBAxx/Include/system_stm32wbaxx.h 	изменено:      stm32cubeide/BluZ_archive/Drivers/CMSIS/Device/ST/STM32WBAxx/LICENSE.txt 	изменено:      stm32cubeide/BluZ_archive/Drivers/CMSIS/Include/cachel1_armv7.h 	изменено:      stm32cubeide/BluZ_archive/Drivers/CMSIS/Include/cmsis_armcc.h 	изменено:      stm32cubeide/BluZ_archive/Drivers/CMSIS/Include/cmsis_armclang.h 	изменено:      stm32cubeide/BluZ_archive/Drivers/CMS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
Routing:
- net GND: track 154.6 -> 164.7 mm
Changed lines of the file:
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@@
+	)
+	(segment
+		(start 81.568056 51.068056)
+		(end 82.797149 51.068056)
+		(width 0.25)
+		(layer "F.Cu")
+		(net 1)
 	)
 	(segment
@@
 	)
 	(segment
+		(start 81.46 50.96)
+		(end 81.568056 51.068056)
+		(width 0.25)
+		(layer "F.Cu")
+		(net 1)
+	)
+	(segment
 		(start 64.057107 44.627107)
 		(end 62.887893 43.457893)
@@
 	)
 	(segment
-		(start 83.151472 51.1)
-		(end 81.6 51.1)
+		(start 83.292124 50.86303)
+		(end 83.469418 50.685736)
 		(width 0.25)
 		(layer "F.Cu")
@@
 	)
 	(segment
-		(start 83.575736 50.924264)
-		(end 83.99 50.51)
-		(width 0.25)
-		(layer "F.Cu")
-		(net 1)
-	)
-	(segment
 		(start 76.18 50)
 		(end 76.817107 50.637107)
@@
 	)
 	(segment
+		(start 83.893682 50.51)
+		(end 83.99 50.51)
+		(width 0.25)
+		(layer "F.Cu")
+		(net 1)
+	)
+	(segment
 		(start 80.34 50.93)
 		(end 81.41 50.93)
@@
 		(start 70.63 47.25)
 		(end 70.63 48.295786)
-		(width 0.25)
-		(layer "F.Cu")
-		(net 1)
-	)
-	(segment
-		(start 81.6 51.1)
-		(end 81.46 50.96)
 		(width 0.25)
 		(layer "F.Cu")
@@
 	)
 	(arc
+		(start 83.292124 50.86303)
+		(mid 83.065028 51.014771)
+		(end 82.797149 51.068056)
+		(width 0.25)
+		(layer "F.Cu")
+		(net 1)
+	)
+	(arc
 		(start 72.207107 50.287107)
 		(mid 72.53153 50.50388)
@@
 	)
 	(arc
-		(start 83.575736 50.924264)
-		(mid 83.381082 51.054328)
-		(end 83.151472 51.1)
-		(width 0.25)
-		(layer "F.Cu")
-		(net 1)
-	)
-	(arc
 		(start 74.422893 50.287107)
 		(mid 74.09847 50.50388)
@@
 		(end 62.887893 43.457893)
 		(width 0.6)
+		(layer "F.Cu")
+		(net 1)
+	)
+	(arc
+		(start 83.893682 50.51)
+		(mid 83.664072 50.555672)
+		(end 83.469418 50.685736)
+		(width 0.25)
 		(layer "F.Cu")
 		(net 1)
@@
 	)
 	(segment
+		(start 74.876494 51.496494)
+		(end 74.71 51.33)
+		(width 0.4)
+		(layer "F.Cu")
+		(net 27)
+	)
+	(segment
+		(start 80.674694 51.595203)
+		(end 80.663853 51.584362)
+		(width 0.4)
+		(layer "F.Cu")
+		(net 27)
+	)
+	(segment
 		(start 73.94 45.58)
 		(end 73.94 45.665736)
@@
 	)
 	(segment
+		(start 84.668553 51.364108)
+		(end 84.566142 51.466519)
+		(width 0.4)
+		(layer "F.Cu")
+		(net 27)
+	)
+	(segment
 		(start 83.252132 49.087868)
 		(end 83.157868 49.182132)
@@
 	)
 	(segment
+		(start 82.186972 51.683071)
+		(end 80.886826 51.683071)
+		(width 0.4)
+		(layer "F.Cu")
+		(net 27)
+	)
+	(segment
 		(start 69.47 48.61)
 		(end 69.27 48.61)
@@
 	)
 	(segment
+		(start 84.212589 51.612965)
+		(end 82.257078 51.612965)
+		(width 0.4)
+		(layer "F.Cu")
+		(net 27)
+	)
+	(segment
 		(start 74.66 42.03)
 		(end 74.66 42.02)
@@
 	)
 	(segment
+		(start 82.257078 51.612965)
+		(end 82.186972 51.683071)
+		(width 0.4)
+		(layer "F.Cu")
+		(net 27)
+	)
+	(segment
 		(start 84.795 50.05)
 		(end 84.684264 50.05)
@@
 		(end 65.911472 38.74)
 		(width 0.5)
+		(layer "F.Cu")
+		(net 27)
+	)
+	(segment
+		(start 80.451721 51.496494)
+		(end 74.876494 51.496494)
+		(width 0.4)
+		(layer "F.Cu")
+		(net 27)
+	)
+	(segment
+		(start 84.815 50.05)
+		(end 84.815 51.010554)
+		(width 0.4)
 		(layer "F.Cu")
 		(net 27)
@@
 	)
 	(segment
-		(start 84.815 50.05)
-		(end 84.815 51.509)
-		(width 0.4)
-		(layer "F.Cu")
-		(net 27)
-	)
-	(segment
 		(start 76.38 41.73)
 		(end 74.96 41.73)
@@
 		(end 66.674264 40.534264)
 		(width 0.5)
+		(layer "F.Cu")
+		(net 27)
+	)
+	(arc
+		(start 84.212589 51.612965)
+		(mid 84.40393 51.574905)
+		(end 84.566142 51.466519)
+		(width 0.4)
 		(layer "F.Cu")
 		(net 27)
@@
 	)
 	(arc
+		(start 80.886826 51.683071)
+		(mid 80.772021 51.660235)
+		(end 80.674694 51.595203)
+		(width 0.4)
+		(layer "F.Cu")
+		(net 27)
+	)
+	(arc
 		(start 67.215686 41.595686)
 		(mid 67.475225 41.769104)
@@
 	)
 	(arc
+		(start 84.815 51.010554)
+		(mid 84.77694 51.201896)
+		(end 84.668553 51.364108)
+		(width 0.4)
+		(layer "F.Cu")
+		(net 27)
+	)
+	(arc
 		(start 78.662893 38.532893)
 		(mid 78.33847 38.31612)
@@
 		(layer "F.Cu")
 		(net 27)
+	)
+	(arc
+		(start 80.663853 51.584362)
+		(mid 80.566526 51.51933)
+		(end 80.451721 51.496494)
+		(width 0.4)
+		(layer "F.Cu")
+		(net 27)
