File: kicad/bluz_v2_typec/bluz_v1.kicad_pcb (KiCad board)
At the start: 2 copper layers, 29.6 x 16.1 mm, 76 parts, among them J10 Conn, J11 Conn, J12 BTAnt, J2 Conn, J3 Conn, J4 Conn, J5 Conn, J6 Conn, J7 Conn, J8 Conn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

Commit message: изменено:      kicad/bluz_v2_typec/bluz_v1.kicad_pcb 	изменено:      kicad/bluz_v2_typec/bom/ibom.html 	изменено:      kicad/bluz_v2_typec/fp-info-cache 	изменено:      stm32cubeide/BluZ_LPM/Core/Inc/main.h 	изменено:      stm32cubeide/BluZ_LPM/Release/BluZ_LPM_v1.elf
Parts:
- R2: moved to B.Cu
- moved C10 5.58 mm to (104.7, 58.1), turned to 90 degrees
- moved R1 4.15 mm to (117.7, 54.0), turned to 180 degrees
- moved C13 4.01 mm to (112.3, 56.8), turned to -90 degrees
- moved R2 2.35 mm to (115.8, 54.0)
- moved R5 1.56 mm to (102.5, 54.4)
- moved J5 1.25 mm to (102.0, 53.2)
- moved C26 1.17 mm to (119.6, 57.4)
- moved C24 1.17 mm to (119.6, 58.4)
- moved J3 1.06 mm to (110.3, 56.9)
- moved R12 1.05 mm to (119.7, 54.4), turned to 0 degrees
- moved Q2 0.98 mm to (120.0, 55.9), turned to -90 degrees
- moved R8 0.93 mm to (111.5, 53.4), turned to -90 degrees
- moved C30 0.68 mm to (105.1, 55.3), turned to 180 degrees
- moved R9 0.61 mm to (110.5, 53.3), turned to -90 degrees
- moved C20 0.45 mm to (100.1, 57.0)
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Routing:
- net batLev: track 13.8 -> 10.3 mm
- net +BATT: track 52.2 -> 50.4 mm
- net cmpAdj: track 6.98 -> 5.50 mm
- net Net-(LED1-+-Pad1): track 10.7 -> 9.32 mm
- net +2V8: track 54.2 -> 55.5 mm
- net GND: track 64.9 -> 65.9 mm, vias 19 -> 20
- net Net-(Q2-D): track 1.84 -> 0.98 mm
- net /swc: track 2.18 -> 2.95 mm
- net LED: track 1.78 -> 2.32 mm

Commit message: изменено:      kicad/bluz_v2_typec/bluz_v1.kicad_pcb 	изменено:      kicad/bluz_v2_typec/bluz_v1.kicad_sch 	изменено:      kicad/bluz_v2_typec/fp-info-cache
Parts:
- L3: value SRN4018-6R8M -> LQH31MN5R6J03L
- moved C18 0.38 mm to (103.6, 48.8)
- moved J12 0.32 mm to (102.5, 47.7)
Routing:
- net GND: track 65.9 -> 75.2 mm, vias 20 -> 21
Changed lines of the file:
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@@
 	(footprint "Capacitor_SMD:C_0402_1005Metric"
 		(layer "B.Cu")
-		(at 103.23339 48.81 180)
+		(at 103.61097 48.81 180)
 		(descr "Capacitor SMD 0402 (1005 Metric), square (rectangular) end terminal, IPC_7351 nominal, (Body size source: IPC-SM-782 page 76, https://www.pcb-3d.com/wordpress/wp-content/uploads/ipc-sm-782a_amendment_1_and_2.pdf), generated with kicad-footprint-generator")
 		(tags "capacitor")
@@
 	(footprint "lib:conn_mini"
 		(layer "B.Cu")
-		(at 102.16 47.71226 180)
+		(at 102.478152 47.68158 180)
 		(property "Reference" "J12"
 			(at 1.76 -0.41 0)
@@
 			)
 		)
-		(property "Value" "SRN4018-6R8M"
+		(property "Value" "LQH31MN5R6J03L"
 			(at 0 -1.83 90)
 			(layer "B.Fab")
@@
 	(segment
 		(start 99.854214 50.44)
-		(end 101.2225 50.44)
+		(end 101.21364 50.44)
 		(width 0.4)
 		(layer "F.Cu")
@@
 	)
 	(segment
+		(start 101.21364 50.44)
+		(end 101.2225 50.44)
+		(width 0.4)
+		(layer "F.Cu")
+		(net 26)
+	)
+	(segment
 		(start 105.79774 50.17226)
 		(end 105.79774 49.101954)
@@
 	)
 	(via
-		(at 104.1 48.71)
+		(at 101.21364 50.44)
+		(size 0.6)
+		(drill 0.3)
+		(layers "F.Cu" "B.Cu")
+		(net 26)
+	)
+	(via
+		(at 104.262933 48.747406)
 		(size 0.6)
 		(drill 0.3)
@@
 	)
 	(segment
+		(start 102.59202 46.43902)
+		(end 102.871324 46.718324)
+		(width 0.2)
+		(layer "B.Cu")
+		(net 26)
+	)
+	(segment
 		(start 108.24 53.92375)
 		(end 108.24 52.23625)
@@
 	)
 	(segment
+		(start 102.59202 46.43902)
+		(end 102.561007 46.43902)
+		(width 0.2)
+		(layer "B.Cu")
+		(net 26)
+	)
+	(segment
 		(start 104.805628 50.74226)
 		(end 106.493128 50.74226)
@@
 	)
 	(segment
+		(start 101.322245 47.92631)
+		(end 101.322245 48.436005)
+		(width 0.2)
+		(layer "B.Cu")
+		(net 26)
+	)
+	(segment
 		(start 104.1 47.37)
 		(end 104.1 48.71)
@@
 	)
 	(segment
+		(start 102.871324 46.718324)
+		(end 103.523 47.37)
+		(width 0.2)
+		(layer "B.Cu")
+		(net 26)
+	)
+	(segment
 		(start 119.60702 50.19)
 		(end 119.60702 50.24465)
@@
 	)
 	(segment
+		(start 102.561007 46.43902)
+		(end 101.497981 47.502046)
+		(width 0.2)
+		(layer "B.Cu")
+		(net 26)
+	)
+	(segment
 		(start 104.805628 50.74226)
 		(end 103.40472 50.74226)
@@
 		(net 26)
 	)
+	(segment
+		(start 96.574688 45.919207)
+		(end 102.072207 45.919207)
+		(width 0.3)
+		(layer "B.Cu")
+		(net 26)
+	)
 	(arc
 		(start 108.897107 55.407107)
@@
 	)
 	(arc
+		(start 101.497981 47.502046)
+		(mid 101.367917 47.6967)
+		(end 101.322245 47.92631)
+		(width 0.2)
+		(layer "B.Cu")
+		(net 26)
+	)
+	(arc
 		(start 102.339924 51.31)
 		(mid 102.569534 51.264328)
@@
 	)
 	(segment
+		(start 103.13097 48.81)
+		(end 103.13097 49.51903)
+		(width 0.2)
+		(layer "B.Cu")
+		(net 51)
+	)
+	(segment
 		(start 104.204392 49.654392)
 		(end 104.177868 49.627868)
@@
 	)
 	(segment
-		(start 102.759878 48.91)
-		(end 102.759878 49.53)
+		(start 103.13097 49.51903)
+		(end 103.11 49.54)
 		(width 0.2)
 		(layer "B.Cu")
