File: kicad/bluz_v1_LED/bluz_v1.kicad_pcb (KiCad board)
At the start: 2 copper layers, 35.2 x 17.1 mm, 100 parts, among them J10 Conn, J11 Conn, J12 BTAnt, J2 Conn, J3 Conn, J4 Conn, J40 LS013B7DH05, J5 Conn, J6 Conn, J7 Conn, J8 Conn, J9 USB_C_Receptacle_PowerOnly_6P, M1 Z3OC1T8219731, Q1 NTA4153NT1G, Q2 RUM002N05, Q3 NTA4153NT1G, Q4 NTA4151PT1G, Q5 NTA4153NT1G, Q6 NTA4153NT1G, U1 MCP73831, U2 REF35180QDBVR, U3 TLV3201AIDCK, U4 AP3015KTR, U6 PAM8904EGPR, U7 TPS627451DSSR, Y1 NX1612SA-32MHz, Y2 NX2012SA-32.768

Commit message: изменено:      Android/BluZ_v2/BluZ/Android/BluZ_LPM/BluZ/src/main/java/ru/starline/bluz/MainActivity.kt 	изменено:      Android/BluZ_v2/BluZ/Android/BluZ_LPM/BluZ/src/main/java/ru/starline/bluz/globalObj.kt 	изменено:      Android/BluZ_v2/BluZ/Android/BluZ_LPM/BluZ/src/main/res/layout-land/activity_main.xml 	изменено:      Android/BluZ_v2/BluZ/Android/BluZ_LPM/BluZ/src/main/res/layout/activity_main.xml 	удалено:       kicad/bluz_v1_LED/bluz_v1-backups/bluz_v1-2026-07-10_154057.zip 	удалено:       kicad/bluz_v1_LED/bluz_v1-backups/bluz_v1-2026-07-10_154720.zip 	удалено:       kicad/bluz_v1_LED/bluz_v1-backups/bluz_v1-2026-07-13_101334.zip 	удалено:       kicad/bluz_v1_LED/bluz_v1-backups/bluz_v1-2026-07-13_113755.zip 	удалено:       kicad/bluz_v1_LED/bluz_v1-backups/bluz_v1-2026-09-14_165340.zip 	удалено:       kicad/bluz_v1_LED/bluz_v1-backups/bluz_v1-2026-09-14_165908.zip 	удалено:       kicad/bluz_v1_LED/bluz_v1-backups/bluz_v1-2026-09-14_170418.zip 	изменено:      kicad/bluz_v1_LED/bluz_v1.kicad_pcb
Parts:
- moved R7 0.71 mm to (101.5, 51.6), turned to 90 degrees
Routing:
- net power_hold: track 2.80 -> 3.46 mm
Other:
- board size 35.2 x 17.1 mm -> 35.2 x 17.9 mm
