File: kicad/bluz_v1_LCD/bluz_lcd_v1.kicad_pcb (KiCad board)
At the start: 2 copper layers, 35.2 x 17.9 mm, 100 parts, among them J10 Conn, J11 Conn, J12 BTAnt, J2 Conn, J3 Conn, J4 Conn, J40 LS013B7DH05, J5 Conn, J6 Conn, J7 Conn, J8 Conn, J9 USB_C_Receptacle_PowerOnly_6P, M1 Z3OC1T8219731, Q1 NTA4153NT1G, Q2 RUM002N05, Q3 NTA4153NT1G, Q4 NTA4151PT1G, Q5 NTA4153NT1G, Q6 NTA4153NT1G, U1 MCP73831, U2 REF35180QDBVR, U3 TLV3201AIDCK, U4 AP3015KTR, U6 PAM8904EGPR, U7 TPS627451DSSR, Y1 NX1612SA-32MHz, Y2 NX2012SA-32.768

Commit message: переименовано: kicad/bluz_v1_LED/2024-05-07_07-39-39.kicad_sym -> kicad/bluz_v1_LCD/2024-05-07_07-39-39.kicad_sym 	переименовано: kicad/bluz_v1_LED/CSPG6_1P05X1P65_STM-L.kicad_mod -> kicad/bluz_v1_LCD/CSPG6_1P05X1P65_STM-L.kicad_mod 	переименовано: kicad/bluz_v1_LED/CSPG6_1P05X1P65_STM-M.kicad_mod -> kicad/bluz_v1_LCD/CSPG6_1P05X1P65_STM-M.kicad_mod 	переименовано: kicad/bluz_v1_LED/CSPG6_1P05X1P65_STM.kicad_mod -> kicad/bluz_v1_LCD/CSPG6_1P05X1P65_STM.kicad_mod 	новый файл:    kicad/bluz_v1_LCD/bluz_lcd_v1-backups/bluz_lcd_v1-2026-10-17_154510.zip 	новый файл:    kicad/bluz_v1_LCD/bluz_lcd_v1-backups/bluz_lcd_v1-2026-10-17_155607.zip 	переименовано: kicad/bluz_v1_LED/bluz_v1.kicad_pcb -> kicad/bluz_v1_LCD/bluz_lcd_v1.kicad_pcb 	переименовано: kicad/bluz_v1_LED/bluz_v1.kicad_prl -> kicad/bluz_v1_LCD/bluz_lcd_v1.kicad_prl 	переименовано: kicad/bluz_v1_LED/bluz_v1.kicad_pro -> kicad/bluz_v1_LCD/bluz_lcd_v1.kicad_pro 	переименовано: kicad/bluz_v1_LED/bluz_v1.kicad_sch -> kicad/bluz_v1_LCD/bluz_lcd_v1.kicad_sch 	переименовано: kicad/bluz_v1_LED/fp-info-cache -> kicad/bluz_v1_LCD/fp-info-cache 	новый файл:    kicad/bluz_v1_LCD/gerber/mill_config.txt 	новый файл:    kicad/bluz_v1_LCD/gerber/mk-gcode.sh 	переименовано: kicad/bluz_v1_LED/gerber/mk-gerber.sh -> kicad/bluz_v1_LCD/gerber/mk-gerber.sh 	удалено:       kicad/bluz_v1_LED/bluz_v1-backups/bluz_v1-2026-09-14_181225.zip 	удалено:       kicad/bluz_v1_LED/bluz_v1-backups/bluz_v1-2026-09-15_141616.zip 	удалено:       kicad/bluz_v1_LED/bluz_v1-backups/bluz_v1-2026-09-15_144107.zip 	удалено:       kicad/bluz_v1_LED/bluz_v1-backups/bluz_v1-2026-09-15_145150.zip 	удалено:       kicad/bluz_v1_LED/bluz_v1-backups/bluz_v1-2026-09-15_150420.zip 	удалено:       kicad/bluz_v1_LED/bluz_v1-backups/bluz_v1-2026-09-15_155235.zip 	удалено:       kicad/bluz_v1_LED/bluz_v1-backups/bluz_v1-2026-09-17_183048.zip 	удалено:       kicad/bluz_v1_LED/bluz_v1-backups/bluz_v1-2026-09-17_183700.zip 	удалено:       kicad/bluz_v1_LED/bluz_v1-backups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
Parts:
- removed C35: 22u, Capacitor_SMD:C_0402_1005Metric
- removed D7: BAS516, Diode_SMD:D_SOD-523
- removed Q6: NTA4153NT1G, Package_TO_SOT_SMD:SOT-723
- removed R22: 5.1M, Resistor_SMD:R_0402_1005Metric
- added R23: 10M, Resistor_SMD:R_0402_1005Metric, B.Cu at (101.6, 50.8)
- C18: moved to F.Cu
- R11, R19: value 5.1M -> 10M
- moved C18 4.53 mm to (104.3, 48.2), turned to 90 degrees
- moved J10 0.84 mm to (100.4, 51.8)
Connections:
- net Rst renamed Net-(D1-RST)
Routing:
- net Net-(D7-K): track 3.05 -> 0.00 mm
- net Net-(Q4-G): track 4.55 -> 2.53 mm, vias 1 -> 0
- net Net-(D1-RST): track 6.60 -> 4.58 mm, vias 2 -> 1
- net (no net): vias 4 -> 0
